File: board/implementation.kicad_sch (KiCad schematic)
At the start: 0 parts

Commit message: initial
Parts:
- added C1: 100nF, Resistor_SMD:R_0603_1608Metric, symbol Device:C_Small
- added R10, R8: 10k, Resistor_SMD:R_0603_1608Metric, symbol Device:R_Small
- added R4, R5, R6, R7: 2.2k, Resistor_SMD:R_0603_1608Metric, symbol Device:R_Small
- added R9: 120R, Resistor_SMD:R_0603_1608Metric, symbol Device:R_Small
- added U1: MAX485E, Package_SO:SO-8_3.9x4.9mm_P1.27mm, symbol Interface_UART:MAX485E
Connections:
- new net 3.3V: C1.1, R4.1, R5.1, R6.1, R7.1, R8.1, U1.8 (VCC)
- new net A: R10.1, R9.2, U1.6 (A)
- new net B: R8.2, R9.1, U1.7 (B)
- new net GND: C1.2, R10.2, U1.5 (GND)
- new net RX: R7.2, U1.1 (RO)
- new net RX_EN: R6.2, U1.2 (~{RE})
- new net TX: R4.2, U1.4 (DI)
- new net TX_EN: R5.2, U1.3 (DE)
